File: katana60-pro-plate.kicad_pcb (KiCad board)
At the start: 2 copper layers, 285 x 94.6 mm, 77 parts

Commit message: - Add readme file - update design - update production files
Parts:
- MX31, MX37_2, MX39_2, MX45: footprint marbastlib-xp-plate-mx:Plate-MP_MX_1.25u -> RominRonin:Plate-MP_MX_1.25u_Katana60_middle_pair
- S3: footprint marbastlib-xp-plate-mx:Plate-MP_MX_7u -> RominRonin:Plate-MP_MX_7u_Katana60_7u_overlapping
- moved REF** 0.79 mm to (206.4, 119.1)
- turned MX39_2 to 180 degrees

Commit message: Finalise plate and exports
Parts:
- REF**: moved to B.Cu
- turned REF** to 180 degrees
- turned S1 to 180 degrees
- turned S2 to 180 degrees
- turned S3 to 180 degrees
Other:
- outline, holes or cut-outs redrawn
