File: katana60-pro-plate.kicad_sch (KiCad schematic)
At the start: 82 parts

Commit message: Finalise plate and exports
Parts:
- removed MX37, MX39, MX65, MX67, MX68, MX69, MX71: MX-NoLED, marbastlib-xp-plate-mx:Plate-MP_MX_1u, symbol MX_Alps_Hybrid:MX-NoLED
Changed lines of the file:
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@@
-    )
-  )
-  (symbol (lib_id "MX_Alps_Hybrid:MX-NoLED") (at 180.34 205.74 0) (unit 1)
-    (in_bom yes) (on_board yes) (dnp no) (fields_autoplaced)
-    (property "Reference" "MX71" (at 181.2256 199.39 0)
-      (effects (font (size 1.524 1.524)))
-    )
-    (property "Value" "MX-NoLED" (at 181.2256 200.66 0)
-      (effects (font (size 0.508 0.508)))
-    )
-    (property "Footprint" "marbastlib-xp-plate-mx:Plate-MP_MX_1u" (at 164.465 206.375 0)
-      (effects (font (size 1.524 1.524)) hide)
-    )
-    (property "Datasheet" "" (at 164.465 206.375 0)
-      (effects (font (size 1.524 1.524)) hide)
-    )
-    (pin "1")
-    (pin "2")
-    (instances
-      (project "katana60-pro-plate"
-        (path "/b3baaebd-c99d-4218-99ba-d40a73031965"
-          (reference "MX71") (unit 1)
-        )
-      )
     )
   )
@@
     )
   )
-  (symbol (lib_id "MX_Alps_Hybrid:MX-NoLED") (at 154.94 129.54 0) (unit 1)
-    (in_bom yes) (on_board yes) (dnp no) (fields_autoplaced)
-    (property "Reference" "MX39" (at 155.8256 123.19 0)
-      (effects (font (size 1.524 1.524)))
-    )
-    (property "Value" "MX-NoLED" (at 155.8256 124.46 0)
-      (effects (font (size 0.508 0.508)))
-    )
-    (property "Footprint" "marbastlib-xp-plate-mx:Plate-MP_MX_1u" (at 139.065 130.175 0)
-      (effects (font (size 1.524 1.524)) hide)
-    )
-    (property "Datasheet" "" (at 139.065 130.175 0)
-      (effects (font (size 1.524 1.524)) hide)
-    )
-    (pin "1")
-    (pin "2")
-    (instances
-      (project "katana60-pro-plate"
-        (path "/b3baaebd-c99d-4218-99ba-d40a73031965"
-          (reference "MX39") (unit 1)
-        )
-      )
-    )
-  )
   (symbol (lib_id "MX_Alps_Hybrid:MX-NoLED") (at 116.84 129.54 0) (unit 1)
     (in_bom yes) (on_board yes) (dnp no) (fields_autoplaced)
@@
         (path "/b3baaebd-c99d-4218-99ba-d40a73031965"
           (reference "H5") (unit 1)
-        )
-      )
-    )
-  )
-  (symbol (lib_id "MX_Alps_Hybrid:MX-NoLED") (at 154.94 205.74 0) (unit 1)
-    (in_bom yes) (on_board yes) (dnp no) (fields_autoplaced)
-    (property "Reference" "MX69" (at 155.8256 199.39 0)
-      (effects (font (size 1.524 1.524)))
-    )
-    (property "Value" "MX-NoLED" (at 155.8256 200.66 0)
-      (effects (font (size 0.508 0.508)))
-    )
-    (property "Footprint" "marbastlib-xp-plate-mx:Plate-MP_MX_1u" (at 139.065 206.375 0)
-      (effects (font (size 1.524 1.524)) hide)
-    )
-    (property "Datasheet" "" (at 139.065 206.375 0)
-      (effects (font (size 1.524 1.524)) hide)
-    )
-    (pin "1")
-    (pin "2")
-    (instances
-      (project "katana60-pro-plate"
-        (path "/b3baaebd-c99d-4218-99ba-d40a73031965"
-          (reference "MX69") (unit 1)
         )
       )
@@
     )
   )
-  (symbol (lib_id "MX_Alps_Hybrid:MX-NoLED") (at 129.54 205.74 0) (unit 1)
-    (in_bom yes) (on_board yes) (dnp no) (fields_autoplaced)
-    (property "Reference" "MX67" (at 130.4256 199.39 0)
-      (effects (font (size 1.524 1.524)))
-    )
-    (property "Value" "MX-NoLED" (at 130.4256 200.66 0)
-      (effects (font (size 0.508 0.508)))
-    )
-    (property "Footprint" "marbastlib-xp-plate-mx:Plate-MP_MX_1u" (at 113.665 206.375 0)
-      (effects (font (size 1.524 1.524)) hide)
-    )
-    (property "Datasheet" "" (at 113.665 206.375 0)
-      (effects (font (size 1.524 1.524)) hide)
-    )
-    (pin "1")
-    (pin "2")
-    (instances
-      (project "katana60-pro-plate"
-        (path "/b3baaebd-c99d-4218-99ba-d40a73031965"
-          (reference "MX67") (unit 1)
-        )
-      )
-    )
-  )
   (symbol (lib_id "MX_Alps_Hybrid:MX-NoLED") (at 66.04 167.64 0) (unit 1)
     (in_bom yes) (on_board yes) (dnp no) (fields_autoplaced)
@@
     )
   )
-  (symbol (lib_id "MX_Alps_Hybrid:MX-NoLED") (at 129.54 129.54 0) (unit 1)
-    (in_bom yes) (on_board yes) (dnp no) (fields_autoplaced)
-    (property "Reference" "MX37" (at 130.4256 123.19 0)
-      (effects (font (size 1.524 1.524)))
-    )
-    (property "Value" "MX-NoLED" (at 130.4256 124.46 0)
-      (effects (font (size 0.508 0.508)))
-    )
-    (property "Footprint" "marbastlib-xp-plate-mx:Plate-MP_MX_1u" (at 113.665 130.175 0)
-      (effects (font (size 1.524 1.524)) hide)
-    )
-    (property "Datasheet" "" (at 113.665 130.175 0)
-      (effects (font (size 1.524 1.524)) hide)
-    )
-    (pin "1")
-    (pin "2")
-    (instances
-      (project "katana60-pro-plate"
-        (path "/b3baaebd-c99d-4218-99ba-d40a73031965"
-          (reference "MX37") (unit 1)
-        )
-      )
-    )
-  )
   (symbol (lib_id "Mechanical:MountingHole") (at 165.1 228.6 0) (unit 1)
     (in_bom yes) (on_board yes) (dnp no) (fields_autoplaced)
@@
         (path "/b3baaebd-c99d-4218-99ba-d40a73031965"
           (reference "MX17") (unit 1)
-        )
-      )
-    )
-  )
-  (symbol (lib_id "MX_Alps_Hybrid:MX-NoLED") (at 142.24 205.74 0) (unit 1)
-    (in_bom yes) (on_board yes) (dnp no) (fields_autoplaced)
-    (property "Reference" "MX68" (at 143.1256 199.39 0)
-      (effects (font (size 1.524 1.524)))
-    )
-    (property "Value" "MX-NoLED" (at 143.1256 200.66 0)
-      (effects (font (size 0.508 0.508)))
-    )
-    (property "Footprint" "marbastlib-xp-plate-mx:Plate-MP_MX_1u" (at 126.365 206.375 0)
-      (effects (font (size 1.524 1.524)) hide)
-    )
-    (property "Datasheet" "" (at 126.365 206.375 0)
-      (effects (font (size 1.524 1.524)) hide)
-    )
-    (pin "1")
-    (pin "2")
-    (instances
-      (project "katana60-pro-plate"
-        (path "/b3baaebd-c99d-4218-99ba-d40a73031965"
-          (reference "MX68") (unit 1)
         )
       )
@@
         )
       )
-    )
-  )
-  (symbol (lib_id "MX_Alps_Hybrid:MX-NoLED") (at 104.14 205.74 0) (unit 1)
-    (in_bom yes) (on_board yes) (dnp no) (fields_autoplaced)
-    (property "Reference" "MX65" (at 105.0256 199.39 0)
-      (effects (font (size 1.524 1.524)))
-    )
-    (property "Value" "MX-NoLED" (at 105.0256 200.66 0)
-      (effects (font (size 0.508 0.508)))
-    )
-    (property "Footprint" "marbastlib-xp-plate-mx:Plate-MP_MX_1u" (at 88.265 206.375 0)
-      (effects (font (size 1.524 1.524)) hide)
-    )
-    (property "Datasheet" "" (at 88.265 206.375 0)
-      (effects (font (size 1.524 1.524)) hide)
-    )
-    (pin "1")
-    (pin "2")
-    (instances
-      (project "katana60-pro-plate"
-        (path "/b3baaebd-c99d-4218-99ba-d40a73031965"
-          (reference "MX65") (unit 1)
-        )
-      )
